File: board/mandreko-deej.kicad_pcb (KiCad board)
At the start: 2 copper layers, 89.5 x 113.5 mm, 26 parts, among them U1 ProMicroC

Commit message: Fixed footprints of sliders, after verifying original was incorrect. Routed wires. Generated fabrication outputs
Parts:
- R1, R2, R3, R4, R5: footprint Bourns:POT_PTA6043 -> Bourns:PTA6043-2015DP-B103
- moved R3 37.0 mm to (152.2, 96.1), turned to 90 degrees
- moved R1 37.0 mm to (118.9, 96.1), turned to 90 degrees
- moved R2 37.0 mm to (135.5, 96.1), turned to 90 degrees
- moved R4 37.0 mm to (168.7, 96.1), turned to 90 degrees
- moved R5 37.0 mm to (185.3, 96.1), turned to 90 degrees
- moved S3 0.09 mm to (152.6, 49.5)
Connections:
- D2 pad 2: unconnected-(D2-DOUT-Pad2) -> Net-(D2-DOUT)
- D3 pad 4: unconnected-(D3-DIN-Pad4) -> Net-(D2-DOUT)
- R1 pad 1: GND -> Net-(R1-Pad1)
- R1 pad 3: Net-(R1-Pad3) -> GND
- R2 pad 1: GND -> Net-(R2-Pad1)
- R2 pad 3: Net-(R2-Pad3) -> GND
- R3 pad 1: GND -> Net-(R3-Pad1)
- R3 pad 3: Net-(R3-Pad3) -> GND
- R4 pad 1: GND -> Net-(R4-Pad1)
- R4 pad 3: Net-(R4-Pad3) -> GND
- R5 pad 1: GND -> Net-(R5-Pad1)
- R5 pad 3: Net-(R5-Pad3) -> GND
- S1 pad 1: Net-(R1-Pad3) -> Net-(R1-Pad1)
- S2 pad 1: Net-(R2-Pad3) -> Net-(R2-Pad1)
- S3 pad 1: Net-(R3-Pad3) -> Net-(R3-Pad1)
- S4 pad 1: Net-(R4-Pad3) -> Net-(R4-Pad1)
- S5 pad 1: Net-(R5-Pad3) -> Net-(R5-Pad1)
Routing:
- net GND: track 12.9 -> 178.3 mm, vias 10 -> 0
- net Net-(R4-Pad1): track 0.00 -> 88.4 mm
- net Net-(R2-Pad1): track 0.00 -> 88.2 mm
- net Net-(R1-Pad1): track 0.00 -> 88.1 mm
- net Net-(R3-Pad1): track 0.00 -> 87.7 mm
- net Net-(R5-Pad1): track 0.00 -> 87.5 mm
- net Net-(R5-Pad3): track 82.4 -> 0.00 mm
- net Net-(R4-Pad3): track 82.4 -> 0.00 mm
- net Net-(R3-Pad3): track 82.4 -> 0.00 mm
- net Net-(R2-Pad3): track 82.4 -> 0.00 mm
- net Net-(R1-Pad3): track 82.4 -> 0.00 mm
- net 5V: track 278.7 -> 305.3 mm
- net Net-(D2-DOUT): track 0.00 -> 22.9 mm
- net A0: track 45.8 -> 55.3 mm
- net A6: track 72.3 -> 80.9 mm
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Other:
- board text added: "Matt Andreko 2024 Deej Board v1.0 https://deej.rocks/"

Commit message: Fixed board wiring error. Regenerated fabrication files. Added PlatformIO project with LED code. Added STEP of the board 3d model.
Connections:
- C1 pad 1: GND -> 5V
- C1 pad 2: 5V -> GND
- C2 pad 1: GND -> 5V
- C2 pad 2: 5V -> GND
- C3 pad 1: GND -> 5V
- C3 pad 2: 5V -> GND
- C4 pad 1: GND -> 5V
- C4 pad 2: 5V -> GND
- C5 pad 1: GND -> 5V
- C5 pad 2: 5V -> GND
- D1 pad 1: GND -> 5V
- D1 pad 3: 5V -> GND
- D2 pad 1: GND -> 5V
- D2 pad 3: 5V -> GND
- D3 pad 1: GND -> 5V
- D3 pad 3: 5V -> GND
- D4 pad 1: GND -> 5V
- D4 pad 3: 5V -> GND
- D5 pad 1: GND -> 5V
- D5 pad 3: 5V -> GND
Routing:
- net GND: track 178.3 -> 12.8 mm, vias 0 -> 10
- net 5V: track 305.3 -> 358.4 mm
- net Net-(R1-Pad1): track 88.1 -> 86.2 mm
- net Net-(R2-Pad1): track 88.2 -> 86.4 mm
- net Net-(R3-Pad1): track 87.7 -> 85.9 mm
- net Net-(R4-Pad1): track 88.4 -> 86.8 mm
- net Net-(R5-Pad1): track 87.5 -> 86.1 mm
- net A0: track 55.3 -> 54.0 mm
- net A2: track 30.5 -> 29.2 mm
- net A3: track 27.2 -> 25.8 mm
- net Net-(D4-DOUT): track 23.7 -> 22.9 mm
Other:
- board text added: "Matt Andreko 2024 Deej Board v1.0 Revision 2 https://deej.rocks/"
- board text removed: "Matt Andreko 2024 Deej Board v1.0 https://deej.rocks/"
